File: MCU datalogger.kicad_pcb (KiCad board)
At the start: 2 copper layers, 0 parts

Commit message: Completed placement of footprints
Parts:
- added BT1: Battery, Connector_PinHeader_2.54mm:PinHeader_1x02_P2.54mm_Vertical, F.Cu at (66.7, 94.0)
- added C1: 0.1uF, Capacitor_SMD:C_0805_2012Metric, F.Cu at (81.6, 88.3)
- added C2: 22pF, Capacitor_SMD:C_0805_2012Metric, F.Cu at (96.2, 104.1)
- added C3: 22pF, Capacitor_SMD:C_0805_2012Metric, F.Cu at (86.0, 88.3)
- added C4: 0.1uF, Capacitor_SMD:C_0805_2012Metric, F.Cu at (96.2, 108.6)
- added C5: 100nF, Capacitor_SMD:C_0805_2012Metric, F.Cu at (90.5, 88.3)
- added D1: LED, LED_SMD:LED_0805_2012Metric, F.Cu at (100.7, 88.9)
- added D2: LED, LED_SMD:LED_0805_2012Metric, F.Cu at (96.2, 88.9)
- added H1: MountingHole, MountingHole:MountingHole_2.1mm, F.Cu at (66.0, 114.3)
- added H2: MountingHole, MountingHole:MountingHole_2.1mm, F.Cu at (66.0, 88.9)
- added H3: MountingHole, MountingHole:MountingHole_2.1mm, F.Cu at (111.8, 88.9)
- added H4: MountingHole, MountingHole:MountingHole_2.1mm, F.Cu at (111.1, 114.3)
- added J1: Conn_01x04_Pin, Connector_PinHeader_2.54mm:PinHeader_1x04_P2.54mm_Vertical, F.Cu at (108.6, 102.2)
- added J2: Conn_01x04_Pin, Connector_PinHeader_2.54mm:PinHeader_1x04_P2.54mm_Vertical, F.Cu at (95.2, 113.0)
- added J3: Conn_01x09_Pin, Connector_PinHeader_2.54mm:PinHeader_1x09_P2.54mm_Vertical, F.Cu at (70.5, 113.0)
- added J4: Conn_02x03_Odd_Even, Connector_PinHeader_2.54mm:PinHeader_2x03_P2.54mm_Vertical, F.Cu at (106.0, 93.3)
- added R1: 10K, Resistor_SMD:R_0805_2012Metric, F.Cu at (72.1, 108.6)
- added R2: 10K, Resistor_SMD:R_0805_2012Metric, F.Cu at (76.5, 108.6)
- added R3: 4.7K, Resistor_SMD:R_0805_2012Metric, F.Cu at (96.2, 99.7)
- added R4: 4.7K, Resistor_SMD:R_0805_2012Metric, F.Cu at (96.3, 95.9)
- added R5: 330, Resistor_SMD:R_0805_2012Metric, F.Cu at (100.6, 92.1)
- added R6: 10K, Resistor_SMD:R_0805_2012Metric, F.Cu at (100.7, 95.9)
- added R7: 330, Resistor_SMD:R_0805_2012Metric, F.Cu at (96.2, 92.1)
- added U1: 24LC1025, Package_SO:SOIC-8_5.3x5.3mm_P1.27mm, F.Cu at (74.3, 90.2)
- added U2: 24LC1025, Package_SO:SOIC-8_5.3x5.3mm_P1.27mm, F.Cu at (74.3, 97.2)
- added U3: DS1337S_, footprints:SOIC127P600X175-8N, F.Cu at (74.3, 104.1)
- added U4: ATMEGA328P-AU, footprints:QFP80P900X900X120-32N, F.Cu at (86.4, 97.2)
- added Y1: 32.768 KHz, Crystal:Crystal_SMD_5032-2Pin_5.0x3.2mm_HandSoldering, F.Cu at (66.7, 104.8)
- added Y2: 16 MHz, Crystal:Crystal_SMD_5032-2Pin_5.0x3.2mm_HandSoldering, F.Cu at (85.7, 106.7)
Other:
- board outline added: 50.8 x 30.5 mm
