File: MCU datalogger.kicad_pcb (KiCad board)
At the start: 2 copper layers, 50.8 x 30.5 mm, 29 parts, among them J1 Conn_01x04_Pin, J2 Conn_01x04_Pin, J3 Conn_01x09_Pin, J4 Conn_02x03_Odd_Even, U1 24LC1025, U2 24LC1025, U3 DS1337S_, U4 ATMEGA328P-AU, Y1 32.768 KHz, Y2 16 MHz

Commit message: Routing and GND Vcc complete
Parts:
- moved U1 7.68 mm to (73.4, 97.8)
- moved U2 7.25 mm to (73.9, 89.9)
- moved J2 2.30 mm to (97.5, 113.3)
- moved R2 1.34 mm to (75.4, 109.4), turned to 180 degrees
- moved U3 1.21 mm to (73.1, 104.3)
- moved BT1 1.14 mm to (65.5, 94.0)
- moved Y2 1.14 mm to (86.9, 106.7), turned to 180 degrees
- moved R1 1.13 mm to (71.3, 109.4), turned to 180 degrees
- moved D1 1.07 mm to (101.6, 88.4)
- moved D2 1.02 mm to (97.1, 88.4), turned to 0 degrees
- moved J1 1.02 mm to (109.6, 102.2)
- moved J4 1.02 mm to (107.1, 93.3)
- moved R5 1.02 mm to (101.6, 92.1)
- moved R6 1.02 mm to (101.7, 95.9)
- moved R7 1.02 mm to (97.2, 92.1)
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Routing:
- net /SCK: track 0.00 -> 108.8 mm, vias 0 -> 3
- net /Vcc: track 0.00 -> 99.8 mm, vias 0 -> 1
- net Net-(BT1-+): track 0.00 -> 65.9 mm, vias 0 -> 5
- net /SDA: track 0.00 -> 60.0 mm, vias 0 -> 2
- net GND: track 0.00 -> 52.5 mm, vias 0 -> 6
- net /TX: track 0.00 -> 36.0 mm, vias 0 -> 1
- net /RX: track 0.00 -> 32.1 mm, vias 0 -> 1
- net Net-(U4-PB7): track 0.00 -> 32.1 mm, vias 0 -> 2
- net Net-(U4-PB6): track 0.00 -> 26.6 mm
- net /RESET: track 0.00 -> 26.4 mm, vias 0 -> 4
- net /D2: track 0.00 -> 26.0 mm, vias 0 -> 1
- net /MOSI: track 0.00 -> 26.0 mm
- net /D3: track 0.00 -> 24.5 mm
- net /MISO: track 0.00 -> 22.1 mm, vias 0 -> 1
- net /D4: track 0.00 -> 21.9 mm
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
Commit message: completed routing
Parts:
- moved J3 0.89 mm to (71.4, 113.3)
- moved H3 0.51 mm to (111.8, 88.9)
- moved H4 0.51 mm to (111.8, 114.3)
- moved BT1 0.25 mm to (65.8, 94.0)
Routing:
- net GND: track 52.5 -> 76.8 mm, vias 6 -> 7
- net /D8: track 17.9 -> 11.9 mm
- net /D7: track 18.4 -> 12.4 mm
- net Net-(U4-PB7): track 32.1 -> 26.7 mm
- net /D2: track 26.0 -> 30.6 mm
- net /D6: track 17.0 -> 13.6 mm
- net /D5: track 16.0 -> 13.9 mm
- net Net-(U4-PB6): track 26.6 -> 25.3 mm
- net /D3: track 24.5 -> 23.2 mm
- net /RX: track 32.1 -> 33.2 mm
- net /Vcc: track 99.8 -> 100.6 mm
- net /D4: track 21.9 -> 21.2 mm
- net /TX: track 36.0 -> 35.5 mm
- added copper zone on F.Cu, net /Vcc
- added copper zone on B.Cu, net GND

Commit message: Completed Design of 2-layer
Parts:
- moved H3 1.66 mm to (110.1, 88.8)
- moved H4 1.20 mm to (110.6, 114.5)
- moved C4 0.99 mm to (97.3, 107.6)
- moved BT1 0.59 mm to (65.8, 94.6)
- moved J3 0.48 mm to (71.6, 113.7)
- moved J2 0.37 mm to (97.6, 113.6)
- moved H2 0.20 mm to (65.8, 88.9)
- moved H1 0.06 mm to (66.0, 114.3)
- renumbered Y2 to Y1, Y1 to Y2
Connections:
- BT1 pad 1: Net-(BT1-+) -> /Vcc
- C5 pad 1: Net-(BT1-+) -> /Vcc
- D2 pad 2: Net-(BT1-+) -> /Vcc
- U4 pad 18: Net-(BT1-+) -> /Vcc
- U4 pad 4: Net-(BT1-+) -> /Vcc
Routing:
- net /Vcc: track 100.6 -> 184.4 mm, vias 1 -> 6
- net Net-(BT1-+): track 66.2 -> 0.00 mm, vias 5 -> 0
- net GND: track 76.8 -> 105.9 mm, vias 7 -> 8
- net /D2: track 30.6 -> 25.8 mm
- net /RESET: track 26.5 -> 25.2 mm
- net Net-(U4-AREF): track 18.5 -> 17.3 mm
- net Net-(U4-PB6): track 25.3 -> 24.2 mm
- net Net-(U3-~{INTA}): track 7.03 -> 7.88 mm
- net Net-(U4-PB7): track 26.7 -> 26.2 mm
Other:
- board size 50.8 x 30.5 mm -> 51.6 x 32.4 mm
- board text added: "2"
- board text added: "2Mbit EEPROM RTC I2C, SPI, GPIO's"
- board text added: "3"
- board text added: "4"
- board text added: "5"
- board text added: "6"
- board text added: "7"
- board text added: "8"
- board text added: "Data Logger with ATMega328P."
- board text added: "GND"
- board text added: "GPIO"
- board text added: "I2C"
- board text added: "ICSP"
- board text added: "ICSP MISO |Vcc SCK |MOSI RESET|GND"
- board text added: "RX"
- board text added: "SCK"
- board text added: "SDA"
- board text added: "SERIAL"
- board text added: "TX"
- board text added: "Vcc"
